Commit message: Friction and damping parameterized

File: lwr_description/model/kuka_lwr.urdf.xacro (robot description, xacro)
@@ -16,4 +16,9 @@
 	<xacro:property name="min_stiffness" value="0"/>
 	<xacro:property name="rate_stiffness" value="20000"/> <!-- reflex to stiffness -->
+<!-- 	<xacro:property name="friction_lwr" value="10"/>
+	<xacro:property name="damping_lwr" value="1.0"/>
+ -->
+ <xacro:property name="friction_lwr" value="2"/>
+	<xacro:property name="damping_lwr" value="0.5"/>
 	<!-- URDF model /-->
 	<xacro:macro name="kuka_lwr" params="parent name *origin">
@@ -51,5 +56,5 @@
 			<axis xyz="0 0 1"/>
 			<limit lower="${-170 * M_PI / 180}" upper="${170 * M_PI / 180}" effort="176" velocity="${velocity_scale * 110 * M_PI / 180}" />
-			<dynamics friction="10.0" damping="1.0"/>
+			<dynamics friction="${friction_lwr}" damping="${damping_lwr}"/>
 			<parent link="${name}_base_link"/>
 			<child link="${name}_1_link"/>
@@ -101,5 +106,5 @@
 			<axis xyz="0 -1 0"/>
 			<limit lower="${-120 * M_PI / 180}" upper="${120 * M_PI / 180}" effort="176" velocity="${velocity_scale * 110 * M_PI / 180}" />
-			<dynamics friction="10.0" damping="1.0"/>
+			<dynamics friction="${friction_lwr}" damping="${damping_lwr}"/>
 			<parent link="${name}_1_link"/>
 			<child link="${name}_2_link"/>
@@ -151,5 +156,5 @@
 			<axis xyz="0 0 1"/>
 			<limit lower="${-170 * M_PI / 180}" upper="${170 * M_PI / 180}" effort="100" velocity="${velocity_scale * 128 * M_PI / 180}" />
-			<dynamics friction="10.0" damping="1.0"/>
+			<dynamics friction="${friction_lwr}" damping="${damping_lwr}"/>
 			<parent link="${name}_2_link"/>
 			<child link="${name}_3_link"/>
@@ -201,5 +206,5 @@
 			<axis xyz="0 1 0"/>
 			<limit lower="${-120 * M_PI / 180}" upper="${120 * M_PI / 180}" effort="100" velocity="${velocity_scale * 128 * M_PI / 180}" />
-			<dynamics friction="10.0" damping="1.0"/>
+			<dynamics friction="${friction_lwr}" damping="${damping_lwr}"/>
 			<parent link="${name}_3_link"/>
 			<child link="${name}_4_link"/>
@@ -251,5 +256,5 @@
 			<axis xyz="0 0 1"/>
 			<limit lower="${-170 * M_PI / 180}" upper="${170 * M_PI / 180}" effort="100" velocity="${velocity_scale * 204 * M_PI / 180}" />
-			<dynamics friction="10.0" damping="1.0"/>
+			<dynamics friction="${friction_lwr}" damping="${damping_lwr}"/>
 			<parent link="${name}_4_link"/>
 			<child link="${name}_5_link"/>
@@ -301,5 +306,5 @@
 			<axis xyz="0 -1 0"/>
 			<limit lower="${-120 * M_PI / 180}" upper="${120 * M_PI / 180}" effort="38" velocity="${velocity_scale * 184 * M_PI / 180}" />
-			<dynamics friction="10.0" damping="1.0"/>
+			<dynamics friction="${friction_lwr}" damping="${damping_lwr}"/>
 			<parent link="${name}_5_link"/>
 			<child link="${name}_6_link"/>
@@ -338,5 +343,5 @@
 			<axis xyz="0 0 1"/>
 			<limit lower="${-170 * M_PI / 180}" upper="${170 * M_PI / 180}" effort="38" velocity="${velocity_scale * 184 * M_PI / 180}" />
-			<dynamics friction="10.0" damping="1.0"/>
+			<dynamics friction="${friction_lwr}" damping="${damping_lwr}"/>
 			<parent link="${name}_6_link"/>
 			<child link="${name}_7_link"/>

Commit message: mb_test

File: lwr_description/model/kuka_lwr.urdf.xacro (robot description, xacro)
@@ -301,10 +301,10 @@
 			<material name="Kuka/DarkGrey"/>
 			</visual>
-			<collision>
+<!-- 			<collision>
 			<origin xyz="0 0 0" rpy="0 0 ${M_PI}"/>
 			<geometry>
 				<cylinder radius="0.04" length="0.05"/>
 			</geometry>
-			</collision>
+			</collision> -->
 		</link>
 		<xacro:kuka_lwr_gazebo name="${name}"/>

Commit message: correcting inertias. To compute inertias we used this tutorial http://gazebosim.org/tutorials?tut=inertia#Mass

File: lwr_description/model/kuka_lwr.urdf.xacro (robot description, xacro)
@@ -16,4 +16,5 @@
 	<xacro:property name="effort_scale" value="1"/>
 	<xacro:property name="use_extra_joints_default" value="true"/>
+	<xacro:property name="inertia_scale" value="10000000"/>
 	<!-- URDF model /-->
 	<xacro:macro name="kuka_lwr" params="parent name *origin use_extra_joints:=${use_extra_joints_default}">
@@ -50,5 +51,5 @@
 			<axis xyz="0 0 1"/>
 			<limit lower="${-170 * M_PI / 180}" upper="${170 * M_PI / 180}" effort="176" velocity="${velocity_scale * 110 * M_PI / 180}" />
-			<dynamics friction="10.0" damping="1.0"/>
+			<dynamics friction="1.0" damping="0.7"/>
 			<parent link="${name}_base_link"/>
 			<child link="${name}_1_link"/>
@@ -57,6 +58,6 @@
 			<inertial>
 				<mass value="${link_mass}"/>
-				<origin rpy="0 0 0" xyz="0 -0.06 0.130"/>
-				<cuboid_inertia_def length="0.12" width="0.06" height="0.260" mass="${link_mass}"/>
+				<origin rpy="0 0 0" xyz="0.00000301 0.02391176 0.11939403"/>
+			    <inertia ixx="${136938.093750 / inertia_scale}" ixy="${4.968005 / inertia_scale}" ixz="${8.730822 / inertia_scale}" iyy="${135390.187500 / inertia_scale}" iyz="${-23715.781250 / inertia_scale}" izz="${40896.656250 / inertia_scale}" />
 			</inertial>
 			<visual>
@@ -91,5 +92,5 @@
 			<axis xyz="0 -1 0"/>
 			<limit lower="${-120 * M_PI / 180}" upper="${120 * M_PI / 180}" effort="176" velocity="${velocity_scale * 110 * M_PI / 180}" />
-			<dynamics friction="10.0" damping="1.0"/>
+			<dynamics friction="1.0" damping="0.7"/>
 			<parent link="${name}_1_link"/>
 			<child link="${name}_2_link"/>
@@ -98,6 +99,6 @@
 			<inertial>
 				<mass value="${link_mass}"/>
-				<origin rpy="0 0 0" xyz="0 0.06 ${0.130 - 0.06}"/>
-				<cuboid_inertia_def length="0.12" width="0.06" height="0.260" mass="${link_mass}"/>
+				<origin rpy="0 0 0" xyz="0.00000301 -0.02391175 0.08110597"/>
+			    <inertia ixx="${136938.093750 / inertia_scale}" ixy="${-4.968005 / inertia_scale}" ixz="${-8.730822 / inertia_scale}" iyy="${135390.187500 / inertia_scale}" iyz="${-23715.781250 / inertia_scale}" izz="${40896.656250 / inertia_scale}" />
 			</inertial>
 			<visual>
@@ -132,5 +133,5 @@
 			<axis xyz="0 0 1"/>
 			<limit lower="${-170 * M_PI / 180}" upper="${170 * M_PI / 180}" effort="100" velocity="${velocity_scale * 128 * M_PI / 180}" />
-			<dynamics friction="10.0" damping="1.0"/>
+			<dynamics friction="1.0" damping="0.7"/>
 			<parent link="${name}_2_link"/>
 			<child link="${name}_3_link"/>
@@ -139,6 +140,6 @@
 			<inertial>
 				<mass value="${link_mass}"/>
-				<origin rpy="0 0 0" xyz="0 0.06 0.130"/>
-				<cuboid_inertia_def length="0.12" width="0.06" height="0.260" mass="${link_mass}"/>
+				<origin rpy="0 0 0" xyz="-0.00000302 -.02391175 0.11939403"/>
+			    <inertia ixx="${136938.093750 / inertia_scale}" ixy="${4.968005 / inertia_scale}" ixz="${-8.730822 / inertia_scale}" iyy="${135390.187500 / inertia_scale}" iyz="${23715.781250 / inertia_scale}" izz="${40896.656250 / inertia_scale}" />
 			</inertial>
 			<visual>
@@ -173,5 +174,5 @@
 			<axis xyz="0 1 0"/>
 			<limit lower="${-120 * M_PI / 180}" upper="${120 * M_PI / 180}" effort="100" velocity="${velocity_scale * 128 * M_PI / 180}" />
-			<dynamics friction="10.0" damping="1.0"/>
+			<dynamics friction="1.0" damping="0.7"/>
 			<parent link="${name}_3_link"/>
 			<child link="${name}_4_link"/>
@@ -180,6 +181,6 @@
 			<inertial>
 				<mass value="${link_mass}"/>
-				<origin rpy="0 0 0" xyz="0 -0.06 ${0.130 - 0.06}"/>
-				<cuboid_inertia_def length="0.12" width="0.06" height="0.2600" mass="${link_mass}"/>
+				<origin rpy="0 0 0" xyz="-0.00000303 .02391175 0.08110597"/>
+			    <inertia ixx="${136938.093750 / inertia_scale}" ixy="${-4.968005 / inertia_scale}" ixz="${8.730822 / inertia_scale}" iyy="${135390.187500 / inertia_scale}" iyz="${23715.781250 / inertia_scale}" izz="${40896.656250 / inertia_scale}" />
 			</inertial>
 			<visual>
@@ -214,5 +215,5 @@
 			<axis xyz="0 0 1"/>
 			<limit lower="${-170 * M_PI / 180}" upper="${170 * M_PI / 180}" effort="100" velocity="${velocity_scale * 204 * M_PI / 180}" />
-			<dynamics friction="10.0" damping="1.0"/>
+			<dynamics friction="1.0" damping="0.7"/>
 			<parent link="${name}_4_link"/>
 			<child link="${name}_5_link"/>
@@ -221,6 +222,6 @@
 			<inertial>
 				<mass value="${link_mass}"/>
-				<origin rpy="0 0 0" xyz="0 0 0.124"/>
-				<cuboid_inertia_def length="0.12" width="0.06" height="0.248" mass="${link_mass}"/>
+				<origin rpy="0 0 0" xyz="-0.00000303 .02391175 0.08110597"/>
+			    <inertia ixx="${82625.953125 / inertia_scale}" ixy="${5.603518 / inertia_scale}" ixz="${8.553005 / inertia_scale}" iyy="${76228.593750 / inertia_scale}" iyz="${-24984.386719 / inertia_scale}" izz="${33607.035156 / inertia_scale}" />
 			</inertial>
 			<visual>
@@ -255,5 +256,5 @@
 			<axis xyz="0 -1 0"/>
 			<limit lower="${-120 * M_PI / 180}" upper="${120 * M_PI / 180}" effort="38" velocity="${velocity_scale * 184 * M_PI / 180}" />
-			<dynamics friction="10.0" damping="1.0"/>
+			<dynamics friction="1.0" damping="0.7"/>
 			<parent link="${name}_5_link"/>
 			<child link="${name}_6_link"/>
@@ -262,6 +263,6 @@
 			<inertial>
 				<mass value="${wrist_mass}"/>
-				<origin rpy="0 0 0" xyz="0 0 0.0625"/>
-				<cuboid_inertia_def length="0.125" width="0.125" height="0.125" mass="${wrist_mass}"/>
+				<origin rpy="0 0 0" xyz="-0.00000001 -.00447585 -0.00290105"/>
+			    <inertia ixx="${29610.587891 / inertia_scale}" ixy="${-0.002319 / inertia_scale}" ixz="${0.023622 / inertia_scale}" iyy="${29691.074219 / inertia_scale}" iyz="${246.776962 / inertia_scale}" izz="${32060.654297 / inertia_scale}" />
 			</inertial>
 			<visual>
@@ -284,5 +285,5 @@
 			<axis xyz="0 0 1"/>
 			<limit lower="${-170 * M_PI / 180}" upper="${170 * M_PI / 180}" effort="38" velocity="${velocity_scale * 184 * M_PI / 180}" />
-			<dynamics friction="10.0" damping="1.0"/>
+			<dynamics friction="1.0" damping="0.7"/>
 			<parent link="${name}_6_link"/>
 			<child link="${name}_7_link"/>
@@ -291,6 +292,6 @@
 			<inertial>
 				<mass value="${tip_mass}"/>
-				<origin xyz="0 0 0"/>
-				<cuboid_inertia_def length="0.1" width="0.1" height="0.1" mass="${tip_mass}"/>
+				<origin rpy="0 0 0" xyz="-0.00000107 0.0 -0.01580145"/>
+			    <inertia ixx="${414.478149 / inertia_scale}" ixy="0.0" ixz="0.0" iyy="${414.478149 / inertia_scale}" iyz="0.0" izz="${694.374329 / inertia_scale}" />
 			</inertial>
 			<visual>
@@ -301,10 +302,10 @@
 			<material name="Kuka/DarkGrey"/>
 			</visual>
-<!-- 			<collision>
-			<origin xyz="0 0 0" rpy="0 0 ${M_PI}"/>
+			<collision>
+			<origin xyz="0 0 -0.005" rpy="0 0 ${M_PI}"/>
 			<geometry>
-				<cylinder radius="0.04" length="0.05"/>
+				<cylinder radius="0.04" length="0.01"/>
 			</geometry>
-			</collision> -->
+			</collision>
 		</link>
 		<xacro:kuka_lwr_gazebo name="${name}"/>

Commit message: Update the inertia of the last link

File: lwr_description/model/kuka_lwr.urdf.xacro (robot description, xacro)
@@ -16,5 +16,5 @@
 	<xacro:property name="effort_scale" value="1"/>
 	<xacro:property name="use_extra_joints_default" value="true"/>
-	<xacro:property name="inertia_scale" value="10000000"/>
+	<xacro:property name="inertia_scale" value="10000000.0"/>
 	<!-- URDF model /-->
 	<xacro:macro name="kuka_lwr" params="parent name *origin use_extra_joints:=${use_extra_joints_default}">
@@ -292,6 +292,8 @@
 			<inertial>
 				<mass value="${tip_mass}"/>
-				<origin rpy="0 0 0" xyz="-0.00000107 0.0 -0.01580145"/>
-			    <inertia ixx="${414.478149 / inertia_scale}" ixy="0.0" ixz="0.0" iyy="${414.478149 / inertia_scale}" iyz="0.0" izz="${694.374329 / inertia_scale}" />
+			    <origin xyz="0 0 -0.014685" rpy="0 0 0"/>
+			    <!-- <inertia ixx="${414.478149 / inertia_scale}" ixy="0.0" ixz="0.0" iyy="${414.478149 / inertia_scale}" iyz="0.0" izz="${694.374329 / inertia_scale}" /> -->
+        		<!-- <inertia ixx="${2 * tip_mass * 0.1 * 0.1 / 5}"  ixy="0"  ixz="0" iyy="${2 * tip_mass * 0.1 * 0.1 / 5}" iyz="0" izz="${2 * tip_mass * 0.1 * 0.1 / 5}" /> -->
+        		<inertia ixx="${1 / 12  * (3 * 0.05 * 0.05 + 0.01 * 0.01)}"  ixy="0"  ixz="0" iyy="${1 / 12  * (3 * 0.05 * 0.05 + 0.01 * 0.01)}" iyz="0" izz="${1 / 12  * (3 * 0.05 * 0.05 + 0.01 * 0.01)}" />
 			</inertial>
 			<visual>
@@ -302,4 +304,5 @@
 			<material name="Kuka/DarkGrey"/>
 			</visual>
+<!--
 			<collision>
 			<origin xyz="0 0 -0.005" rpy="0 0 ${M_PI}"/>
@@ -307,5 +310,5 @@
 				<cylinder radius="0.04" length="0.01"/>
 			</geometry>
-			</collision>
+			</collision> -->
 		</link>
 		<xacro:kuka_lwr_gazebo name="${name}"/>
